File: hardware/breakout_xrt83l30/breakout_xrt83l30.kicad_pcb (KiCad board)
At the start: 4 copper layers, 109 x 46 mm, 36 parts, among them J1 Conn_01x04, J2 Conn_01x05, J3 Conn_01x20, J4 Conn_02x20_Odd_Even, J5 Conn_01x04, J6 Conn_02x20_Odd_Even, J7 Conn_01x20, J8 RJ45, U1 XRT83L30, U2 RClamp3304NA

Commit message: Update/apply XRT83L30 breakout schematic license and release dates.
Other:
- board text added: "XRT83L30 Breakout 20190722 ShareBrained Technology, Inc. Licensed under CERN-OHL-P v2"
- board text removed: "ShareBrained Technology, Inc. XRT83L30 Breakout 20190722"
