File: hardware/tedium_x8/tedium_x8.kicad_pcb (KiCad board)
At the start: 4 copper layers, 96 x 70 mm, 283 parts, among them CON1 BARREL_JACK, J1 Conn_02x20_Odd_Even, J3 DNP, J5 Conn_ARM_JTAG_SWD_10, P1 USB_C, P2 USB_C, Q1 BC817, Q2 Q_PMOS_GSD, Q3 Q_PMOS_GSD, U1 LFE5U-85F-8BG381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

Commit message: HW: Tedium X8: Update symbols, footprints, KiCAD to 5.99-now.
Other:
- net class Default removed
